File: Hardware/Mrk 0 - Prototype/ComboSensorBreakout.brd (EAGLE design)
At the start: 17.8 x 15.7 mm, 13 parts, among them J1 CONN_42.54_SCREW, Q1 DMG3404, U1 SPG30, U2 SHTC3DFN, U3 TPS7A0518DBV, U4 TXS0102DCU

Commit message: Updated/generated BoMs if not present
Parts:
- C5, C6: value (none) -> 0.1uF
Routing:
- net GND: track 43.8 -> 44.3 mm
